File: dicio-sensor/DicioWRK.brd (EAGLE design)
At the start: 58.4 x 90.2 mm, 62 parts, among them J1 WTB-2, J2 WTB-2, J3 JMP2, J4 JMP2, J5 JMP2, J6 WTB-2, J7 TERM10, Q1 BSS84, Q2 BSS84, Q3 BSS84, Q4 BSS84, Q5 BSS84, U1 78MM6610+PSU, U2 APDS-9005, U3 MCP9700, U4 DK-1A-L2-3, U5 RAC01-3.3, U9 MCP3202

Commit message: Working on Rev. 2.
Parts:
- removed J3, J4, J5: JMP2, TORO:JMP2
- U9: value MCP3202 -> MCP3202SOIC; device TORO:MSOP-8[MCP3202] -> TORO:SOIC8
- moved R1 49.1 mm to (3.49, 49.5), turned to 180 degrees
- moved R17 48.5 mm to (8.57, 39.4), turned to 0 degrees
- moved R18 47.9 mm to (8.57, 49.5), turned to 0 degrees
- moved R16 47.6 mm to (3.49, 39.4), turned to 180 degrees
- moved D1 44.3 mm to (2.54, 53.3), turned to 270 degrees
- moved C8 44.1 mm to (88.9, 71.8)
- moved C3 44.1 mm to (86.4, 77.5)
- moved R12 44.1 mm to (86.4, 74.9)
- moved R23 44.1 mm to (86.4, 80.0)
- moved U2 44.1 mm to (86.4, 72.4)
- moved R25 44.1 mm to (78.7, 59.7)
- moved R26 44.1 mm to (78.7, 62.2)
- moved R27 44.1 mm to (78.7, 64.8)
- moved Q3 43.0 mm to (6.35, 53.3), turned to 90 degrees
- moved Q4 42.7 mm to (6.35, 43.2), turned to 90 degrees
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Connections:
- removed net AIP: C16.1, C17.1, R15.1, R7.1, U4.P$4
- removed net N$12: J5.P$1, Q5.1, R19.1
- removed net N$2: J3.P$1, Q3.1, R18.1
- removed net N$6: J4.P$1, Q4.1, R17.1
- new net N$8: R15.1, U4.P$3
- net !BUTTON!: now also Q5.1, R19.1; no longer J5.P$2
- net !C1_EN!: now also Q3.1, R18.1; no longer J3.P$2
- net !C2_EN!: now also Q4.1, R17.1; no longer J4.P$2
- net NOUT: now also U4.P$4; no longer R15.2
- net VACN: now also C16.1, C17.1, R15.2, R7.1; no longer U4.P$3
Routing:
- net AIP: track 59.6 -> 0.00 mm, vias 12 -> 0
- net VDD: track 76.7 -> 30.6 mm, vias 38 -> 1
- net MISO: track 56.8 -> 10.7 mm, vias 3 -> 0
- net !CS_PWR!: track 55.8 -> 13.7 mm
- net !C2_EN!: track 52.0 -> 14.8 mm
- net VACN: track 0.00 -> 35.6 mm, vias 9 -> 0
- net MOSI: track 49.4 -> 14.4 mm, vias 0 -> 2
- net SCLK: track 43.7 -> 10.4 mm, vias 1 -> 0
- net !ALARM!: track 40.7 -> 9.84 mm
- net !CS_SENSE!: track 29.2 -> 0.00 mm
- net !FAULT!: track 26.6 -> 0.00 mm, vias 2 -> 0
- net !BUTTON!: track 48.3 -> 21.9 mm
- net NOUT: track 85.7 -> 59.9 mm, vias 10 -> 1
- net !C1_EN!: track 50.0 -> 27.5 mm
- net C2: track 9.46 -> 21.7 mm
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- added copper zone on layer 1, net N$8
- removed copper zone on layer 1, net AIP
- removed copper zone on layer 16, net AIP
- removed copper zone on layer 1, net GND
- removed copper zone on layer 16, net NOUT
- removed copper zone on layer 16, net VACN
- removed copper zone on layer 16, net VDD
Other:
- board size 58.4 x 90.2 mm -> 106.7 x 90.2 mm
- board text removed: "BUTTON"
- board text removed: "COIL2"

Commit message: Dicio sensor Rev 1
Parts:
- removed R12: 3.3k, resistor:R0805
- added R6: 10k, resistor:R0805
- U2: value APDS-9005 -> TSL250RD; device TORO:APDS-9005 -> TORO:SOIC8
- moved J6 82.9 mm to (78.7, 36.8)
- moved D3 64.1 mm to (64.8, 48.3), turned to 180 degrees
- moved C3 62.1 mm to (63.5, 19.7), turned to 270 degrees
- moved Q5 61.4 mm to (64.8, 44.5), turned to 0 degrees
- moved C8 60.2 mm to (45.1, 30.5)
- moved R20 58.8 mm to (61.0, 47.3), turned to 90 degrees
- moved R22 57.3 mm to (63.8, 39.4), turned to 90 degrees
- moved R21 57.0 mm to (64.8, 35.9), turned to 0 degrees
- moved U2 56.9 mm to (58.4, 22.9), turned to 0 degrees
- moved R19 55.2 mm to (61.0, 42.2), turned to 270 degrees
- moved C14 54.5 mm to (64.1, 30.5), turned to 0 degrees
- moved C13 54.1 mm to (64.1, 27.9), turned to 0 degrees
- moved D1 52.3 mm to (54.6, 48.3), turned to 180 degrees
- moved J7 51.7 mm to (78.7, 8.89)
- moved J1 51.2 mm to (3.81, 20.3)
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Connections:
- removed net !ALARM!: J7.P$2, U1.7
- removed net !FAULT!: J7.P$1, U1.5
- removed net S_LIGHT: C3.1, R12.2, U2.6, U9.2
- new net N$6: R6.2, U2.7, U9.2
- net !C1_EN!: now also J7.P$9; no longer J7.P$8
- net !C2_EN!: now also J7.P$8; no longer J7.P$9
- net !CS_PWR!: now also J7.P$3, R25.1; no longer J7.P$6, R24.1
- net GND: now also J7.P$2, R6.1, U2.4; no longer R12.1
- net MISO: now also J7.P$5, R27.1; no longer J7.P$4, R26.1
- net MOSI: now also J7.P$6, R24.1; no longer J7.P$5, R27.1
- net SCLK: now also J7.P$4, R26.1; no longer J7.P$3, R25.1
- net VDD: now also C3.1, J7.P$1, U2.6; no longer U2.1
Routing:
- net MISO: track 10.7 -> 64.2 mm, vias 0 -> 1
- net SCLK: track 10.4 -> 62.8 mm, vias 0 -> 1
- net MOSI: track 14.4 -> 62.6 mm
- net !C2_EN!: track 14.8 -> 56.3 mm, vias 0 -> 1
- net !CS_SENSE!: track 0.00 -> 38.2 mm, vias 0 -> 1
- net !C1_EN!: track 27.5 -> 57.7 mm, vias 0 -> 3
- net !CS_PWR!: track 13.7 -> 39.8 mm, vias 0 -> 1
- net N$6: track 0.00 -> 19.7 mm
- net !BUTTON!: track 21.9 -> 40.4 mm, vias 0 -> 1
- net S_LIGHT: track 10.5 -> 0.00 mm
- net !ALARM!: track 9.84 -> 0.00 mm
- net S_TEMP: track 12.2 -> 19.0 mm
- net GND: track 39.5 -> 42.7 mm, vias 14 -> 18
- net N$10: track 0.00 -> 2.86 mm
- net VDD: track 30.6 -> 28.6 mm, vias 1 -> 0
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Other:
- board size 106.7 x 90.2 mm -> 82.5 x 50.8 mm
- board text added: "/BTN"
- board text added: "/C1"
- board text added: "/C2"
- board text added: "/CSP"
- board text added: "/CSS"
- board text added: "0xD1C10001"
- board text added: "BTN"
- board text added: "DICIO SENSOR"
- board text added: "DSANTORO. 0x10433900."
- board text added: "GND"
- board text added: "MISO"
- board text added: "MOSI"
- board text added: "SCLK"
- board text added: "VACL"
- board text added: "VACN"
- board text added: "VDD"
- board text removed: "BUTTON IN"
- board text removed: "DICIO SENSOR BOARD"
- board text removed: "FIREFLY CONNECT"
- board text removed: "LIN"
- board text removed: "NIN"
- board text removed: "Rev. 0."
- board text removed: "[th3b1g]toro. 0x0339."

Commit message: R1-Out for Fab.
Parts:
- moved J1 9.16 mm to (8.89, 27.9), turned to 180 degrees
- moved C3 2.62 mm to (61.0, 20.3), turned to 0 degrees
- moved C13 2.54 mm to (61.6, 27.9)
- moved C14 2.54 mm to (61.6, 30.5)
- moved D2 2.54 mm to (41.9, 48.3)
- moved Q4 2.54 mm to (41.9, 44.5)
- moved R24 2.54 mm to (68.6, 34.9)
- moved R26 2.54 mm to (63.5, 12.7)
- moved U9 2.54 mm to (50.8, 34.3)
- moved R13 2.54 mm to (31.1, 43.2)
- moved R14 2.54 mm to (31.1, 39.1)
- moved C1 2.54 mm to (57.1, 14.6)
- moved C10 2.54 mm to (45.7, 14.0)
- moved C11 2.54 mm to (43.2, 14.0)
- moved C12 2.54 mm to (40.6, 14.0)
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Routing:
- net SCLK: track 62.8 -> 60.3 mm
- net !CS_PWR!: track 39.8 -> 38.2 mm
- net VACN: track 36.8 -> 35.6 mm
- net MOSI: track 62.6 -> 61.5 mm
Other:
- board size 82.5 x 50.8 mm -> 80 x 50.8 mm
