File: dicio-sensor/DicioWRK.sch (EAGLE design)
At the start: 62 parts, among them J1 WTB-2, J2 WTB-2, J3 JMP2, J4 JMP2, J5 JMP2, J6 WTB-2, J7 TERM10, Q1 BSS84, Q2 BSS84, Q3 BSS84, Q4 BSS84, Q5 BSS84, U1 78MM6610+PSU, U2 APDS-9005, U3 MCP9700, U4 DK-1A-L2-3, U5 RAC01-3.3, U9 MCP3202

Commit message: Working on Rev. 2.
Parts:
- removed J3, J4, J5: JMP2, TORO:JMP2
- U9: value MCP3202 -> MCP3202SOIC; device TORO:MCP3202 -> TORO:MCP3202SOIC
Connections:
- removed net AIP: C16.1, C17.1, R15.1, R7.1, U4.LOAD-
- removed net N$12: J5.1, Q5.G, R19.1
- removed net N$2: J3.1, Q3.G, R18.1
- removed net N$6: J4.1, Q4.G, R17.1
- new net N$8: R15.1, U4.LOAD+
- net !BUTTON!: now also Q5.G, R19.1; no longer J5.P$2
- net !C1_EN!: now also Q3.G, R18.1; no longer J3.P$2
- net !C2_EN!: now also Q4.G, R17.1; no longer J4.P$2
- net NOUT: now also U4.LOAD-; no longer R15.2
- net VACN: now also C16.1, C17.1, R15.2, R7.1; no longer U4.LOAD+
Other:
- moved on the sheet: R15

Commit message: Dicio sensor Rev 1
Parts:
- R6: value 3.3k -> 10k; DKPN 311-3.30KCRCT-ND -> 311-10KARCT-ND
- U2: value APDS-9005 -> TSL250RD; device TORO:APDS-9005 -> TORO:TSL250RD; DKPN 516-1717-1-ND -> (none)
- renumbered R12 to R6
Connections:
- removed net !ALARM!: J7.P$2, U1.!ACCRIT!
- removed net !FAULT!: J7.P$1, U1.!ACFAULT!
- removed net S_LIGHT: C3.1, R6.2, U2.ROUT, U9.CH0
- new net N$6: R6.2, U2.OUT, U9.CH0
- net !C1_EN!: now also J7.P$9; no longer J7.P$8
- net !C2_EN!: now also J7.P$8; no longer J7.P$9
- net !CS_PWR!: now also J7.P$3, R25.1; no longer J7.P$6, R24.1
- net GND: now also J7.P$2, U2.GND
- net MISO: now also J7.P$5, R27.1; no longer J7.P$4, R26.1
- net MOSI: now also J7.P$6, R24.1; no longer J7.P$5, R27.1
- net SCLK: now also J7.P$4, R26.1; no longer J7.P$3, R25.1
- net VDD: now also C3.1, J7.P$1
Other:
- moved on the sheet: C3, R23, R24, R25, R26, R27

Commit message: R1-Out for Fab.
Changed lines of the file:
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@@
 <net name="!C1_EN!" class="0">
-<segment>
-<wire x1="40.64" y1="50.8" x2="30.48" y2="50.8" width="0.1524" layer="91"/>
-<label x="30.48" y="50.8" size="1.778" layer="95"/>
-</segment>
 <segment>
 <pinref part="R14" gate="G$1" pin="1"/>
@@
 <wire x1="45.72" y1="50.8" x2="43.18" y2="50.8" width="0.1524" layer="91"/>
 <pinref part="R18" gate="G$1" pin="1"/>
-<wire x1="43.18" y1="50.8" x2="40.64" y2="50.8" width="0.1524" layer="91"/>
+<wire x1="43.18" y1="50.8" x2="33.02" y2="50.8" width="0.1524" layer="91"/>
 <wire x1="43.18" y1="50.8" x2="43.18" y2="53.34" width="0.1524" layer="91"/>
 <junction x="43.18" y="50.8"/>
+<label x="33.02" y="50.8" size="1.778" layer="95"/>
 </segment>
 <segment>
@@
 </net>
 <net name="!C2_EN!" class="0">
-<segment>
-<wire x1="86.36" y1="50.8" x2="76.2" y2="50.8" width="0.1524" layer="91"/>
-<label x="76.2" y="50.8" size="1.778" layer="95"/>
-</segment>
 <segment>
 <pinref part="R13" gate="G$1" pin="1"/>
@@
 <pinref part="R17" gate="G$1" pin="1"/>
 <wire x1="88.9" y1="53.34" x2="88.9" y2="50.8" width="0.1524" layer="91"/>
-<wire x1="88.9" y1="50.8" x2="86.36" y2="50.8" width="0.1524" layer="91"/>
+<wire x1="88.9" y1="50.8" x2="76.2" y2="50.8" width="0.1524" layer="91"/>
 <pinref part="Q4" gate="G$1" pin="G"/>
 <wire x1="91.44" y1="50.8" x2="88.9" y2="50.8" width="0.1524" layer="91"/>
 <junction x="88.9" y="50.8"/>
+<label x="76.2" y="50.8" size="1.778" layer="95"/>
 </segment>
 <segment>
@@
 <net name="!BUTTON!" class="0">
 <segment>
-<wire x1="132.08" y1="50.8" x2="121.92" y2="50.8" width="0.1524" layer="91"/>
-<label x="121.92" y="50.8" size="1.778" layer="95"/>
-</segment>
-<segment>
 <pinref part="R22" gate="G$1" pin="2"/>
 <pinref part="C13" gate="G$1" pin="1"/>
@@
 <wire x1="137.16" y1="50.8" x2="134.62" y2="50.8" width="0.1524" layer="91"/>
 <wire x1="134.62" y1="50.8" x2="134.62" y2="53.34" width="0.1524" layer="91"/>
-<wire x1="134.62" y1="50.8" x2="132.08" y2="50.8" width="0.1524" layer="91"/>
+<wire x1="134.62" y1="50.8" x2="121.92" y2="50.8" width="0.1524" layer="91"/>
 <junction x="134.62" y="50.8"/>
+<label x="121.92" y="50.8" size="1.778" layer="95"/>
 </segment>
 </net>
 <net name="N$1" class="0">
 <segment>
-<pinref part="R4" gate="G$1" pin="1"/>
-<wire x1="71.12" y1="157.48" x2="71.12" y2="162.56" width="0.1524" layer="91"/>
-<pinref part="R3" gate="G$1" pin="2"/>
-<wire x1="71.12" y1="162.56" x2="50.8" y2="162.56" width="0.1524" layer="91"/>
 <pinref part="U1" gate="G$1" pin="AVP"/>
-<wire x1="71.12" y1="162.56" x2="81.28" y2="162.56" width="0.1524" layer="91"/>
-<junction x="71.12" y="162.56"/>
 <wire x1="81.28" y1="162.56" x2="91.44" y2="162.56" width="0.1524" layer="91"/>
 <wire x1="91.44" y1="162.56" x2="101.6" y2="162.56" width="0.1524" layer="91"/>
@@
 <pinref part="C4" gate="G$1" pin="1"/>
 <wire x1="81.28" y1="157.48" x2="81.28" y2="162.56" width="0.1524" layer="91"/>
+<pinref part="R4" gate="G$1" pin="1"/>
+<wire x1="71.12" y1="157.48" x2="71.12" y2="162.56" width="0.1524" layer="91"/>
+<wire x1="71.12" y1="162.56" x2="81.28" y2="162.56" width="0.1524" layer="91"/>
 <junction x="81.28" y="162.56"/>
+<pinref part="R3" gate="G$1" pin="2"/>
+<wire x1="71.12" y1="162.56" x2="50.8" y2="162.56" width="0.1524" layer="91"/>
+<junction x="71.12" y="162.56"/>
 </segment>
 </net>
@@
 </segment>
 </net>
-<net name="N$9" class="0">
-<segment>
-<wire x1="71.12" y1="162.56" x2="73.66" y2="162.56" width="0.1524" layer="91"/>
-</segment>
-</net>
